File: pcb/swerve/swerve1/swerve1.kicad_pcb (KiCad board)
At the start: 2 copper layers, 29.2 x 58.4 mm, 7 parts, among them J1 M20-7810645R, J2 M20-7810645R

Commit message: osh version
Parts:
- added R1: 8K2, Resistor_SMD:R_0805_2012Metric_Pad1.20x1.40mm_HandSolder, F.Cu at (79.0, 63.5)
- added R2: 3K, Resistor_SMD:R_0805_2012Metric_Pad1.20x1.40mm_HandSolder, F.Cu at (84.1, 63.5)
- renumbered ADC to ADC1, GPS to GPS1, USFS to IMU1, Motor to Motor1, PMW to PMW1
Connections:
- ADC1 pad 1: Net-(J1-Pad3) -> Net-(ADC1-Pad1)
Routing:
- net Net-(ADC1-Pad1): track 0.00 -> 18.4 mm, vias 0 -> 2
- net Net-(ADC1-Pad4): track 127.3 -> 131.1 mm
- net Net-(J2-Pad8): track 24.1 -> 22.8 mm
- net Net-(ADC1-Pad2): track 24.3 -> 23.2 mm
