File: pcb/swerve/swerve1/swerve1.kicad_pcb (KiCad board)
At the start: 2 copper layers, 29.2 x 58.4 mm, 9 parts, among them J1 M20-7810645R, J2 M20-7810645R

Commit message: updated pcb
Parts:
- added Spare1: BM06B-SRSS-TBLFSN, footprints:CONN_BM06B-SRSS-TB_JST, F.Cu at (72.4, 89.5)
Connections:
- J1 pad 5: unconnected-(J1-Pad5) -> Net-(J1-Pad5)
- J1 pad 6: unconnected-(J1-Pad6) -> Net-(J1-Pad6)
- J1 pad 7: unconnected-(J1-Pad7) -> Net-(J1-Pad7)
- J1 pad 8: unconnected-(J1-Pad8) -> Net-(J1-Pad8)
Routing:
- net Net-(GPS1-Pad2): track 50.7 -> 22.4 mm, vias 0 -> 2
- net Net-(J1-Pad5): track 0.00 -> 28.2 mm, vias 0 -> 2
- net Net-(J1-Pad7): track 0.00 -> 28.2 mm, vias 0 -> 2
- net Net-(J1-Pad8): track 0.00 -> 24.5 mm, vias 0 -> 4
- net Net-(J1-Pad6): track 0.00 -> 22.4 mm, vias 0 -> 4
- net Net-(GPS1-Pad1): track 44.4 -> 33.2 mm, vias 0 -> 2
- net Net-(IMU1-Pad3): track 96.8 -> 87.7 mm, vias 5 -> 7
- net Net-(ADC1-Pad4): track 131.1 -> 139.3 mm, vias 0 -> 2
- net Net-(J2-Pad3): track 28.8 -> 21.8 mm
- net Net-(J2-Pad7): track 35.9 -> 30.7 mm, vias 0 -> 2
- net Net-(ADC1-Pad3): track 47.2 -> 51.2 mm, vias 2 -> 4
- net Net-(J1-Pad3): track 33.5 -> 30.0 mm
- net Net-(IMU1-Pad2): track 34.1 -> 31.5 mm
- net Net-(ADC1-Pad2): track 23.2 -> 21.7 mm
- net Net-(J2-Pad9): track 28.0 -> 26.7 mm
Other:
- board size 29.2 x 58.4 mm -> 25.4 x 61 mm
