File: pcb/swerve/swerve1/swerve1.kicad_sch (KiCad schematic)
At the start: 7 parts, among them J1 M20-7810645R, J2 M20-7810645R, J3 BM04B-SRSS-TBT LFSN, J4 BM04B-SRSS-TBT LFSN, J5 BM04B-SRSS-TBT LFSN, J6 BM06B-SRSS-TBLFSN, J7 BM04B-SRSS-TBT LFSN

Commit message: osh version
Parts:
- added R1: 8K2, Resistor_SMD:R_0805_2012Metric_Pad1.20x1.40mm_HandSolder, symbol Device:R_Small_US
- added R2: 3K, Resistor_SMD:R_0805_2012Metric_Pad1.20x1.40mm_HandSolder, symbol Device:R_Small_US
- renumbered J7 to ADC1, J3 to GPS1, J4 to IMU1, J5 to Motor1, J6 to PMW1
Connections:
- net at ADC1.4, GPS1.4, IMU1.4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: now also R2.2
- net at J1.3: now also R1.2, R2.1; no longer ADC1.1
- new net: ADC1.1, R1.1

Commit message: updated pcb
Parts:
- added Spare1: BM06B-SRSS-TBLFSN, CONN_BM06B-SRSS-TB_JST, symbol 2023-07-16_19-21-55:BM06B-SRSS-TBLFSN
Connections:
- net at ADC1.4, GPS1.4, IMU1.4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: now also Spare1.6
- net at ADC1.3, GPS1.3, J1.1: now also Spare1.1
- net at J1.5: now also Spare1.4
- net at J1.6: now also Spare1.3
- net at J1.7: now also Spare1.5
- net at J1.8: now also Spare1.2
Changed lines of the file:
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@@
   (junction (at 86.36 59.69) (diameter 0) (color 0 0 0 0)
   )
+  (junction (at 104.14 41.91) (diameter 0) (color 0 0 0 0)
+  )
   (junction (at 139.7 74.93) (diameter 0) (color 0 0 0 0)
   )
@@
   (junction (at 31.75 30.48) (diameter 0) (color 0 0 0 0)
   )
+  (junction (at 86.36 144.78) (diameter 0) (color 0 0 0 0)
+  )
   (junction (at 139.7 59.69) (diameter 0) (color 0 0 0 0)
   )
   (junction (at 139.7 44.45) (diameter 0) (color 0 0 0 0)
   )
+  (wire (pts (xy 78.74 54.61) (xy 90.17 54.61))
+    (stroke (width 0) (type default))
+  )
   (wire (pts (xy 78.74 119.38) (xy 86.36 119.38))
     (stroke (width 0) (type default))
@@
     (stroke (width 0) (type default))
   )
+  (wire (pts (xy 118.11 175.26) (xy 44.45 175.26))
+    (stroke (width 0) (type default))
+  )
   (wire (pts (xy 218.44 104.14) (xy 139.7 104.14))
     (stroke (width 0) (type default))
@@
     (stroke (width 0) (type default))
   )
+  (wire (pts (xy 78.74 52.07) (xy 97.79 52.07))
+    (stroke (width 0) (type default))
+  )
   (wire (pts (xy 55.88 116.84) (xy 46.99 116.84))
     (stroke (width 0) (type default))
   )
+  (wire (pts (xy 90.17 167.64) (xy 118.11 167.64))
+    (stroke (width 0) (type default))
+  )
   (wire (pts (xy 139.7 44.45) (xy 139.7 59.69))
     (stroke (width 0) (type default))
@@
     (stroke (width 0) (type default))
   )
+  (wire (pts (xy 97.79 52.07) (xy 97.79 170.18))
+    (stroke (width 0) (type default))
+  )
   (wire (pts (xy 170.18 83.82) (xy 170.18 99.06))
     (stroke (width 0) (type default))
@@
     (stroke (width 0) (type default))
   )
+  (wire (pts (xy 90.17 54.61) (xy 90.17 167.64))
+    (stroke (width 0) (type default))
+  )
+  (wire (pts (xy 44.45 54.61) (xy 55.88 54.61))
+    (stroke (width 0) (type default))
+  )
   (wire (pts (xy 177.8 139.7) (xy 217.17 139.7))
     (stroke (width 0) (type default))
@@
     (stroke (width 0) (type default))
   )
+  (wire (pts (xy 118.11 172.72) (xy 50.8 172.72))
+    (stroke (width 0) (type default))
+  )
   (wire (pts (xy 38.1 109.22) (xy 38.1 83.82))
     (stroke (width 0) (type default))
@@
     (stroke (width 0) (type default))
   )
+  (wire (pts (xy 104.14 165.1) (xy 104.14 41.91))
+    (stroke (width 0) (type default))
+  )
   (wire (pts (xy 184.15 57.15) (xy 184.15 39.37))
     (stroke (width 0) (type default))
   )
+  (wire (pts (xy 50.8 52.07) (xy 55.88 52.07))
+    (stroke (width 0) (type default))
+  )
   (wire (pts (xy 158.75 33.02) (xy 139.7 33.02))
     (stroke (width 0) (type default))
   )
-  (wire (pts (xy 218.44 41.91) (xy 96.52 41.91))
+  (wire (pts (xy 218.44 41.91) (xy 104.14 41.91))
     (stroke (width 0) (type default))
   )
@@
     (stroke (width 0) (type default))
   )
+  (wire (pts (xy 50.8 52.07) (xy 50.8 172.72))
+    (stroke (width 0) (type default))
+  )
   (wire (pts (xy 158.75 30.48) (xy 96.52 30.48))
     (stroke (width 0) (type default))
@@
     (stroke (width 0) (type default))
   )
+  (wire (pts (xy 118.11 177.8) (xy 86.36 177.8))
+    (stroke (width 0) (type default))
+  )
+  (wire (pts (xy 118.11 165.1) (xy 104.14 165.1))
+    (stroke (width 0) (type default))
+  )
+  (wire (pts (xy 86.36 177.8) (xy 86.36 144.78))
+    (stroke (width 0) (type default))
+  )
   (wire (pts (xy 100.33 101.6) (xy 184.15 101.6))
     (stroke (width 0) (type default))
@@
     (stroke (width 0) (type default))
   )
+  (wire (pts (xy 97.79 170.18) (xy 118.11 170.18))
+    (stroke (width 0) (type default))
+  )
   (wire (pts (xy 158.75 96.52) (xy 218.44 96.52))
     (stroke (width 0) (type default))
@@
     (stroke (width 0) (type default))
   )
+  (wire (pts (xy 104.14 41.91) (xy 96.52 41.91))
+    (stroke (width 0) (type default))
+  )
   (wire (pts (xy 184.15 39.37) (xy 218.44 39.37))
     (stroke (width 0) (type default))
@@
   )
   (wire (pts (xy 124.46 27.94) (xy 158.75 27.94))
+    (stroke (width 0) (type default))
+  )
+  (wire (pts (xy 44.45 54.61) (xy 44.45 175.26))
     (stroke (width 0) (type default))
   )
@@
         )
       )
+    )
+  )
+  (symbol (lib_id "2023-07-16_19-21-55:BM06B-SRSS-TBLFSN") (at 118.11 165.1 0) (unit 1)
+    (in_bom yes) (on_board yes) (dnp no) (fields_autoplaced)
+    (property "Reference" "Spare1" (at 132.08 170.18 0)
+      (effects (font (size 1.524 1.524)) (justify left))
+    )
+    (property "Value" "BM06B-SRSS-TBLFSN" (at 132.08 172.72 0)
+      (effects (font (size 1.524 1.524)) (justify left))
+    )
+    (property "Footprint" "CONN_BM06B-SRSS-TB_JST" (at 118.11 165.1 0)
+      (effects (font (size 1.27 1.27) italic) hide)
+    )
+    (property "Datasheet" "BM06B-SRSS-TBLFSN" (at 118.11 165.1 0)
+      (effects (font (size 1.27 1.27) italic) hide)
+    )
+    (pin "1")
+    (pin "2")
+    (pin "3")
+    (pin "4")
+    (pin "5")
+    (pin "6")
+    (instances
+      (project "swerve1"
+        (path "/2af824b0-300a-497f-aa60-c6e7d89f7305"
+          (reference "Spare1") (unit 1)
+        )
+      )
