File: pcb/swerve/swerve.kicad_sch (KiCad schematic)
At the start: 7 parts, among them J1 SHF-105-01-L-D-SM, J2 SHF-105-01-L-D-SM, J3 SHF-105-01-L-D-SM, J4 SHF-105-01-L-D-SM, J5 BM05B-SRSS-TBLFSN, J6 M20-7810645R, J7 M20-7810645R

Commit message: update pcb
Parts:
- added BLE1, BRE1, FLE1, FRE1: B4B-PH-SM4-TB, Connector_JST:JST_PH_B4B-PH-SM4-TB_1x04-1MP_P2.00mm_Vertical, symbol 2023-07-18_18-49-26:B4B-PH-SM4-TB
- added Cell1: BM03B-SRSS-TBLFSN, CONN_BM03B-SRSS-TBLFSN_JST, symbol 2023-07-26_03-04-05:BM03B-SRSS-TBLFSN
- renumbered J4 to BL1, J3 to BR1, J2 to FL1, J1 to FR1, J5 to Radio1
Connections:
- net at BL1.10, BR1.10, FL1.10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: now also BLE1.1, BRE1.1, Cell1.1, FLE1.1, FRE1.1
- net at BL1.02, BR1.02, FL1.02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: now also Cell1.2
- net at J7.4, Radio1.3: now also Cell1.3
- net at J6.1: now also FLE1.2, FRE1.2
- net at J6.3: now also FLE1.4
- net at J6.4: now also FLE1.3
- net at J6.5: now also FRE1.4
- net at J6.6: now also FRE1.3
- net at J7.1: now also BLE1.2, BRE1.2
- net at J7.10: now also BRE1.4
- net at J7.7: now also BLE1.3
- net at J7.8: now also BLE1.4
- net at J7.9: now also BRE1.3
