File: pcb/swerve/swerve.kicad_pcb (KiCad board)
At the start: 2 copper layers, 47 x 49.5 mm, 7 parts, among them J6 M20-7810645R, J7 M20-7810645R

Commit message: update pcb
Parts:
- added BLE1: B4B-PH-SM4-TB, Connector_JST:JST_PH_B4B-PH-SM4-TB_1x04-1MP_P2.00mm_Vertical, F.Cu at (116.1, 62.7)
- added BRE1: B4B-PH-SM4-TB, Connector_JST:JST_PH_B4B-PH-SM4-TB_1x04-1MP_P2.00mm_Vertical, F.Cu at (105.9, 62.7)
- added Cell1: BM03B-SRSS-TBLFSN, footprints1:CONN_BM03B-SRSS-TBLFSN_JST, F.Cu at (108.2, 76.4)
- added FLE1: B4B-PH-SM4-TB, Connector_JST:JST_PH_B4B-PH-SM4-TB_1x04-1MP_P2.00mm_Vertical, F.Cu at (116.4, 38.9)
- added FRE1: B4B-PH-SM4-TB, Connector_JST:JST_PH_B4B-PH-SM4-TB_1x04-1MP_P2.00mm_Vertical, F.Cu at (106.2, 38.9)
- renumbered FR to BL1, BR to BR1, FL to FL1, BL to FR1, Radio to Radio1
Connections:
- J6 pad 1: unconnected-(J6-Pad1) -> Net-(FLE1-Pad2)
- J6 pad 3: unconnected-(J6-Pad3) -> Net-(FLE1-Pad4)
- J6 pad 4: unconnected-(J6-Pad4) -> Net-(FLE1-Pad3)
- J6 pad 5: unconnected-(J6-Pad5) -> Net-(FRE1-Pad4)
- J6 pad 6: unconnected-(J6-Pad6) -> Net-(FRE1-Pad3)
- J7 pad 1: unconnected-(J7-Pad1) -> Net-(BLE1-Pad2)
- J7 pad 10: unconnected-(J7-Pad10) -> Net-(BRE1-Pad4)
- J7 pad 7: unconnected-(J7-Pad7) -> Net-(BLE1-Pad3)
- J7 pad 8: unconnected-(J7-Pad8) -> Net-(BLE1-Pad4)
- J7 pad 9: unconnected-(J7-Pad9) -> Net-(BRE1-Pad3)
Routing:
- net Net-(BL1-Pad10): track 189.8 -> 303.4 mm, vias 2 -> 5
- net Net-(FLE1-Pad2): track 0.00 -> 100.5 mm, vias 0 -> 2
- net Net-(FLE1-Pad4): track 0.00 -> 80.1 mm, vias 0 -> 2
- net Net-(BLE1-Pad2): track 0.00 -> 73.8 mm, vias 0 -> 2
- net Net-(FLE1-Pad3): track 0.00 -> 73.7 mm, vias 0 -> 4
- net Net-(BLE1-Pad3): track 0.00 -> 72.3 mm, vias 0 -> 2
- net Net-(BLE1-Pad4): track 0.00 -> 60.6 mm, vias 0 -> 2
- net Net-(BRE1-Pad3): track 0.00 -> 58.6 mm, vias 0 -> 2
- net Net-(FRE1-Pad4): track 0.00 -> 57.8 mm, vias 0 -> 4
- net Net-(FRE1-Pad3): track 0.00 -> 47.5 mm, vias 0 -> 2
- net Net-(BRE1-Pad4): track 0.00 -> 46.1 mm, vias 0 -> 2
- net Net-(BL1-Pad02): track 143.7 -> 157.1 mm, vias 10 -> 8
- net Net-(J7-Pad3): track 48.2 -> 61.0 mm, vias 2 -> 4
- net Net-(Cell1-Pad3): track 38.5 -> 48.9 mm
- net Net-(BR1-Pad09): track 39.2 -> 33.7 mm
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Other:
- board size 47 x 49.5 mm -> 68.6 x 49.5 mm

Commit message: updated pcb
Routing:
- net unconnected-(J7-Pad6): track 0.00 -> 13.2 mm, vias 0 -> 3
Changed lines of the file:
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@@
   (segment (start 78.74 77.47) (end 83.82 77.47) (width 0.25) (layer "B.Cu") (net 34))
   (segment (start 90.17 77.47) (end 83.82 77.47) (width 0.25) (layer "B.Cu") (net 34))
+  (segment (start 69.85 66.04) (end 69.85 63.555) (width 0.25) (layer "F.Cu") (net 35))
+  (segment (start 62.6 68.58) (end 64.77 68.58) (width 0.25) (layer "F.Cu") (net 35))
+  (segment (start 64.77 68.58) (end 66.04 69.85) (width 0.25) (layer "F.Cu") (net 35))
+  (segment (start 69.85 63.555) (end 69.85 62.23) (width 0.25) (layer "F.Cu") (net 35))
+  (via (at 66.04 69.85) (size 0.8) (drill 0.4) (layers "F.Cu" "B.Cu") (net 35))
+  (via (at 69.85 62.23) (size 0.8) (drill 0.4) (layers "F.Cu" "B.Cu") (net 35))
+  (via (at 69.85 66.04) (size 0.8) (drill 0.4) (layers "F.Cu" "B.Cu") (net 35))
+  (segment (start 66.04 69.85) (end 69.85 66.04) (width 0.25) (layer "B.Cu") (net 35))
   (segment (start 95.0916 76.2) (end 88.9 76.2) (width 0.25) (layer "F.Cu") (net 36))
   (segment (start 95.846499 76.2) (end 95.0916 76.2) (width 0.25) (layer "F.Cu") (net 36))
